File: pcb-cycling-controller.kicad_sch (KiCad schematic)
At the start: 48 parts, among them J1 Power, J2 USB, J3 PROG, Q1 SI2301CDS-T1-GE3-ES, Q2 SI2301CDS-T1-GE3-ES, SW1 SS12F44G4, U3 AMS1117-5.0, U4 TX4113

Commit message: Rev1 as ordered
Parts:
- C38: JLCPCB Part # C21122 -> (none); LCSC Part # (none) -> C21122
- D3, D4: JLCPCB C7588055 -> (none); LCSC Part # (none) -> C7588055
- F1: LCSC C883153 -> (none)
- J1: LCSC Part # C30436 -> C722717
- J2: LCSC Part # (none) -> C165948
- U4: JLCPCB C5382729 -> (none); LCSC Part # (none) -> C5382729
